File: adapter/active-3/active3-rpi-hub75-adapter.kicad_sch (KiCad schematic)
At the start: 20 parts, among them P1 CONN_02X20, P2 +5V, P4 GND, U1 74HCT245, U2 74HCT245, U3 74HCT245, U4 Reflective IR sensor

Commit message: newer schematics
Parts:
- removed C3: 100n, Capacitor_SMD:C_0805_2012Metric, symbol Device:C
- removed C5: 22u, Capacitor_THT:CP_Radial_D6.3mm_P2.50mm, symbol active3-rpi-hub75-adapter-rescue:CP_Small-Device
- removed C6: 22u, Capacitor_SMD:C_1206_3216Metric, symbol Device:C_Small
- removed P2: +5V, Pin_Headers:Pin_Header_Straight_1x01, symbol Connector_Generic:Conn_01x01
- removed P4: GND, Pin_Headers:Pin_Header_Straight_1x01, symbol Connector_Generic:Conn_01x01
- removed Panel-2: CONN_02X08, Connector_IDC:IDC-Header_2x08_P2.54mm_Vertical, symbol Connector_Generic:Conn_02x08_Odd_Even
- removed U3: 74HCT245, Package_SO:SOIC-20W_7.5x12.8mm_P1.27mm, symbol 74xx:74HC245
- added J1: IR_Sensor_Socket, Connector_PinSocket_2.54mm:PinSocket_1x04_P2.54mm_Horizontal, symbol Connector:Conn_01x04_Socket
- added R5: 10k, Resistor_THT:R_Axial_DIN0207_L6.3mm_D2.5mm_P7.62mm_Horizontal, symbol Device:R_US
- added R6: 470, Resistor_THT:R_Axial_DIN0207_L6.3mm_D2.5mm_P7.62mm_Horizontal, symbol Device:R_US
- added R7: 20k, Resistor_THT:R_Axial_DIN0207_L6.3mm_D2.5mm_P7.62mm_Horizontal, symbol Device:R_US
- C1, C2: footprint Capacitor_SMD:C_0805_2012Metric -> Capacitor_SMD:C_1210_3225Metric
- FID1, FID2: now not fitted
- P1: footprint Pin_Headers:Pin_Header_Straight_2x20 -> Connector_PinSocket_2.54mm:PinSocket_2x20_P2.54mm_Vertical
- Panel-1: footprint Connector_IDC:IDC-Header_2x08_P2.54mm_Vertical -> Connector_PinSocket_2.54mm:PinSocket_2x08_P2.54mm_Horizontal
- R1: footprint Resistor_SMD:R_0805_2012Metric -> Resistor_THT:R_Axial_DIN0207_L6.3mm_D2.5mm_P7.62mm_Horizontal
- R2, R3, R4, U4: now not fitted; now left out of the parts list
Connections:
- net gnd is gone; now on net GND: P1.30 (Pin_30), P1.9 (Pin_9)
- net GND: now also J1.2 (Pin_2), J1.3 (Pin_3), R7.1
- net VCC: now also R5.1, R6.2
- net spin_sync: now also J1.4 (Pin_4), R5.2, R7.2
- net strobe: no longer U2.4 (A2)
- net strobe_buff_1: no longer names the net of U2.16 (B2)
- new net: J1.1 (Pin_1), R6.1
Other:
- note removed: "C alt. footprint"
- note removed: "Pi Power 5V"
